File: sonde xilinx.kicad_sch (KiCad schematic)
At the start: 25 parts, among them J1 DB25MALE, J2 DB9MALE, P1 CONN_6, U1 74LS125, U2 74LS125

Commit message: update to kicad 9
Parts:
- C1: symbol sonde_xilinx_schlib:CP -> sonde_xilinx:CP
- C2, C3, C4, C5: symbol sonde_xilinx_schlib:C -> sonde_xilinx:C
- D1, D2: symbol sonde_xilinx_schlib:DIODESCH -> sonde_xilinx:DIODESCH
- J1: symbol sonde_xilinx_schlib:DB25 -> sonde_xilinx:DB25
- J2: symbol sonde_xilinx_schlib:DB9 -> sonde_xilinx:DB9
- P1: symbol sonde_xilinx_schlib:CONN_6 -> sonde_xilinx:CONN_6
- R1, R10, R11, R12, R13, R14, R2, R4, R5, R6, R7, R8, R9: symbol sonde_xilinx_schlib:R -> sonde_xilinx:R
- U1: symbol sonde_xilinx_schlib:74LS125 -> sonde_xilinx:74LS125_1
- U1: symbol sonde_xilinx_schlib:74LS125 -> sonde_xilinx:74LS125_6
- U1: symbol sonde_xilinx_schlib:74LS125 -> sonde_xilinx:74LS125_7
- U1: symbol sonde_xilinx_schlib:74LS125 -> sonde_xilinx:74LS125
- U2: symbol sonde_xilinx_schlib:74LS125 -> sonde_xilinx:74LS125_2
- U2: symbol sonde_xilinx_schlib:74LS125 -> sonde_xilinx:74LS125_3
- U2: symbol sonde_xilinx_schlib:74LS125 -> sonde_xilinx:74LS125_4
- U2: symbol sonde_xilinx_schlib:74LS125 -> sonde_xilinx:74LS125_5
